Commit message: robot standing

File: install/human_urdf/share/human_urdf/urdf/human_gazebo.xacro (robot description, xacro)
@@ -1,4 +1,4 @@
 <?xml version="1.0"?>
-<robot name="RobPrincewill" xmlns:xacro="http://ros.org/wiki/xacro">
+<robot name="human_urdf" xmlns:xacro="http://ros.org/wiki/xacro">
     <gazebo>
         <xacro:if value="$(arg is_ignition)">
@@ -13,3 +13,43 @@
         </xacro:unless>
     </gazebo>
+    <gazebo reference="camera_left_link">
+  <sensor name="left_eye_camera" type="camera">
+    <always_on>true</always_on>
+    <update_rate>30</update_rate>
+    <visualize>true</visualize>
+    <topic>left_camera/image_raw</topic>
+    <camera>
+      <horizontal_fov>1.047</horizontal_fov>
+      <image>
+        <width>640</width>
+        <height>480</height>
+        <format>R8G8B8</format>
+      </image>
+      <clip>
+        <near>0.05</near>
+        <far>50.0</far>
+      </clip>
+    </camera>
+  </sensor>
+</gazebo>
+<gazebo reference="camera_right_link">
+  <sensor name="right_eye_camera" type="camera">
+    <always_on>true</always_on>
+    <update_rate>30</update_rate>
+    <visualize>true</visualize>
+    <topic>right_camera/image_raw</topic>
+    <camera>
+      <horizontal_fov>1.047</horizontal_fov>
+      <image>
+        <width>640</width>
+        <height>480</height>
+        <format>R8G8B8</format>
+      </image>
+      <clip>
+        <near>0.05</near>
+        <far>50.0</far>
+      </clip>
+    </camera>
+  </sensor>
+</gazebo>
 </robot>

File: src/human_urdf/urdf/human_ros2_control.xacro (robot description, xacro)
@@ -1,5 +1,5 @@
 <?xml version="1.0"?>
-<robot xmlns:xacro="http://www.ros.org/wiki/xacro" name="RobPrincewill">
-    <ros2_control type="system" name="RobPrincewill">
+<robot xmlns:xacro="http://www.ros.org/wiki/xacro" name="human_urdf">
+    <ros2_control type="system" name="human_urdf">
         <!-- Gazebo hardware interface -->
         <hardware>
@@ -80,5 +80,5 @@
                 <!-- Left leg                 -->
         <!-- ========================= -->
-        <joint name="joint_wasitL">
+        <joint name="joint_waistL">
             <command_interface name="position">
                 <param name="min">-1.5708</param>
