Commit message: walking

File: install/human_urdf/share/human_urdf/urdf/human_gazebo.xacro (robot description, xacro)
@@ -1,55 +1 @@
-<?xml version="1.0"?>
-<robot name="human_urdf" xmlns:xacro="http://ros.org/wiki/xacro">
-    <gazebo>
-        <xacro:if value="$(arg is_ignition)">
-            <plugin filename="ign_ros2_control-system" name="ign_ros2_control::IgnitionROS2ControlPlugin">
-                <parameters>$(find human_controller)/config/human_controllers.yaml</parameters>
-            </plugin>
-        </xacro:if>
-        <xacro:unless value="$(arg is_ignition)">
-            <plugin filename="gz_ros2_control-system" name="gz_ros2_control::GazeboSimROS2ControlPlugin">
-                <parameters>$(find human_controller)/config/human_controllers.yaml</parameters>
-            </plugin>
-        </xacro:unless>
-    </gazebo>
-    <gazebo reference="camera_left_link">
-  <sensor name="left_eye_camera" type="camera">
-    <always_on>true</always_on>
-    <update_rate>30</update_rate>
-    <visualize>true</visualize>
-    <topic>left_camera/image_raw</topic>
-    <camera>
-      <horizontal_fov>1.047</horizontal_fov>
-      <image>
-        <width>640</width>
-        <height>480</height>
-        <format>R8G8B8</format>
-      </image>
-      <clip>
-        <near>0.05</near>
-        <far>50.0</far>
-      </clip>
-    </camera>
-  </sensor>
-</gazebo>
-<gazebo reference="camera_right_link">
-  <sensor name="right_eye_camera" type="camera">
-    <always_on>true</always_on>
-    <update_rate>30</update_rate>
-    <visualize>true</visualize>
-    <topic>right_camera/image_raw</topic>
-    <camera>
-      <horizontal_fov>1.047</horizontal_fov>
-      <image>
-        <width>640</width>
-        <height>480</height>
-        <format>R8G8B8</format>
-      </image>
-      <clip>
-        <near>0.05</near>
-        <far>50.0</far>
-      </clip>
-    </camera>
-  </sensor>
-</gazebo>
-</robot>
+/mnt/c/Users/Administrator/Documents/Mechanical/Humaniod/src/human_urdf/urdf/human_gazebo.xacro

File: install/human_urdf/share/human_urdf/urdf/human_ros2_control.xacro (robot description, xacro)
@@ -1,102 +1 @@
-<?xml version="1.0"?>
-<robot xmlns:xacro="http://www.ros.org/wiki/xacro" name="human_urdf">
-    <ros2_control type="system" name="human_urdf">
-        <!-- Gazebo hardware interface -->
-        <hardware>
-            <plugin>gz_ros2_control/GazeboSimSystem</plugin>
-        </hardware>
-        <!-- ========================= -->
-                <!-- RIGHT ARM                 -->
-        <!-- ========================= -->
-        <joint name="joint_shoulderR">
-            <command_interface name="position">
-                <param name="min">-1.5708</param>
-                <param name="max">1.5708</param>
-            </command_interface>
-            <state_interface name="position"/>
-            <state_interface name="velocity"/>
-        </joint>
-        <joint name="joint_elbowR">
-            <command_interface name="position">
-                <param name="min">-0.875</param>
-                <param name="max">1.5708</param>
-            </command_interface>
-            <state_interface name="position"/>
-            <state_interface name="velocity"/>
-        </joint>
-        <!-- ========================= -->
-                <!-- Left ARM                 -->
-        <!-- ========================= -->
-        <joint name="joint_shoulderL">
-            <command_interface name="position">
-                <param name="min">-1.5708</param>
-                <param name="max">1.5708</param>
-            </command_interface>
-            <state_interface name="position"/>
-            <state_interface name="velocity"/>
-        </joint>
-        <joint name="joint_elbowL">
-            <command_interface name="position">
-                <param name="min">-0.942</param>
-                <param name="max">1.5708</param>
-            </command_interface>
-            <state_interface name="position"/>
-            <state_interface name="velocity"/>
-        </joint>
-        <!-- ========================= -->
-                <!-- Neck                 -->
-        <!-- ========================= -->
-        <joint name="joint_neck">
-            <command_interface name="position">
-                <param name="min">-1.5708</param>
-                <param name="max">1.5708</param>
-            </command_interface>
-            <state_interface name="position"/>
-            <state_interface name="velocity"/>
-        </joint>
-        <!-- ========================= -->
-                <!-- Right Leg                 -->
-        <!-- ========================= -->
-        <joint name="joint_waistR">
-            <command_interface name="position">
-                <param name="min">-1.5708</param>
-                <param name="max">1.5708</param>
-            </command_interface>
-            <state_interface name="position"/>
-            <state_interface name="velocity"/>
-        </joint>
-        <!-- ========================= -->
-                <!-- Right Knee                 -->
-        <!-- ========================= -->
-        <joint name="joint_kneeR">
-            <command_interface name="position">
-                <param name="min">-1.5708</param>
-                <param name="max">0.75</param>
-            </command_interface>
-            <state_interface name="position"/>
-            <state_interface name="velocity"/>
-        </joint>
-        <!-- ========================= -->
-                <!-- Left leg                 -->
-        <!-- ========================= -->
-        <joint name="joint_waistL">
-            <command_interface name="position">
-                <param name="min">-1.5708</param>
-                <param name="max">1.5708</param>
-            </command_interface>
-            <state_interface name="position"/>
-            <state_interface name="velocity"/>
-        </joint>
-        <!-- ========================= -->
-                <!-- Left KNEE               -->
-        <!-- ========================= -->
-        <joint name="joint_kneeL">
-            <command_interface name="position">
-                <param name="min">-0.2</param>
-                <param name="max">1.5708</param>
-            </command_interface>
-            <state_interface name="position"/>
-            <state_interface name="velocity"/>
-        </joint>
-    </ros2_control>
-</robot>
+/mnt/c/Users/Administrator/Documents/Mechanical/Humaniod/src/human_urdf/urdf/human_ros2_control.xacro

File: install/human_urdf/share/human_urdf/urdf/human_urdf.urdf.xacro (robot description, xacro)
@@ -1,557 +1 @@
-<?xml version="1.0"?>
-<robot
-  name="human_urdf"
-  xmlns:xacro="http://ros.org/wiki/xacro">
-  <!-- Start GZ or Ignition depending on ROS 2 Version -->
-  <xacro:arg name="is_ignition" default="true"/>
-  <!-- Load simulated or Real Hardware Interfaces -->
-  <xacro:arg name="is_sim" default="true"/>
-  <!-- Include Gazebo Parameters -->
-  <xacro:include filename="$(find human_urdf)/urdf/human_gazebo.xacro" />
-  <!-- Include ros2_control Plugins -->
-  <xacro:include filename="$(find human_urdf)/urdf/human_ros2_control.xacro" />
-  <!-- ============================================================ -->
-  <!-- BASE FOOTPRINT                                                -->
-  <!-- ============================================================ -->
-  <link name="base_footprint"/>
-  <joint name="base_footprint_joint" type="fixed">
-    <parent link="base_footprint"/>
-    <child link="base_link"/>
-    <origin xyz="0 0 0.8" rpy="3.14159 0 0"/>
-  </joint>
-  <!-- ============================================================ -->
-  <!-- BASE LINK                                                      -->
-  <!-- ============================================================ -->
-  <link name="base_link">
-    <inertial>
-      <origin
-        xyz="6.1619E-07 0.025013 0.0081305"
-        rpy="0 0 0" />
-      <mass value="4.6092" />
-      <inertia
-        ixx="0.041497"
-        ixy="-9.5688E-09"
-        ixz="2.9922E-07"
-        iyy="0.071384"
-        iyz="-9.7456E-06"
-        izz="0.03187" />
-    </inertial>
-    <visual>
-      <origin
-        xyz="0 0 0"
-        rpy="0 0 0" />
-      <geometry>
-        <mesh
-          filename="package://human_urdf/meshes/base_link.STL"
-          scale="10.0 10.0 10.0"/>
-      </geometry>
-      <material name="">
-        <color rgba="0.79216 0.81961 0.93333 1" />
-      </material>
-    </visual>
-    <collision>
-      <origin
-        xyz="0 0 0"
-        rpy="0 0 0" />
-      <geometry>
-        <mesh
-          filename="package://human_urdf/meshes/base_link.STL"
-          scale="10.0 10.0 10.0"/>
-      </geometry>
-    </collision>
-  </link>
-  <!-- ============================================================ -->
-  <!-- RIGHT SHOULDER                                                 -->
-  <!-- ============================================================ -->
-  <link name="shoulderR_link">
-    <inertial>
-      <origin
-        xyz="0.0037883 -0.092283 0.064976"
-        rpy="0 0 0" />
-      <mass value="0.43205" />
-      <inertia
-        ixx="0.001734"
-        ixy="1.263E-05"
-        ixz="-8.2186E-05"
-        iyy="0.0015347"
-        iyz="0.00021665"
-        izz="0.0003291" />
-    </inertial>
-    <visual>
-      <origin xyz="0 0 0" rpy="0 0 0" />
-      <geometry>
-        <mesh
-          filename="package://human_urdf/meshes/shoulderR_link.STL"
-          scale="10.0 10.0 10.0"/>
-      </geometry>
-      <material name="">
-        <color rgba="0.79216 0.81961 0.93333 1" />
-      </material>
-    </visual>
-    <collision>
-      <origin xyz="0 0 0" rpy="0 0 0" />
-      <geometry>
-        <mesh
-          filename="package://human_urdf/meshes/shoulderR_link.STL"
-          scale="10.0 10.0 10.0"/>
-      </geometry>
-    </collision>
-  </link>
-  <joint name="joint_shoulderR" type="revolute">
-    <origin
-      xyz="0.077756 0.025 -0.13145"
-      rpy="0 0 1.5708" />
-    <parent link="base_link"/>
-    <child link="shoulderR_link"/>
-    <axis xyz="0 1 0"/>
-    <limit
-      lower="-1.5708"
-      upper="1.5708"
-      effort="10"
-      velocity="5" />
-  </joint>
-  <!-- ============================================================ -->
-  <!-- RIGHT ELBOW                                                    -->
-  <!-- ============================================================ -->
-  <link name="elbowR_link">
-    <inertial>
-      <origin
-        xyz="-0.10086 -0.015 -0.10143"
-        rpy="0 0 0" />
-      <mass value="0.47524" />
-      <inertia
-        ixx="0.0012989"
-        ixy="-2.2731E-12"
-        ixz="-0.0011482"
-        iyy="0.0024409"
-        iyz="8.351E-13"
-        izz="0.0012859" />
-    </inertial>
-    <visual>
-      <origin xyz="0 0 0" rpy="0 0 0" />
-      <geometry>
-        <mesh
-          filename="package://human_urdf/meshes/elbowR_link.STL"
-          scale="10.0 10.0 10.0"/>
-      </geometry>
-      <material name="">
-        <color rgba="0.79216 0.81961 0.93333 1" />
-      </material>
-    </visual>
-    <collision>
-      <origin xyz="0 0 0" rpy="0 0 0" />
-      <geometry>
-        <mesh
-          filename="package://human_urdf/meshes/elbowR_link.STL"
-          scale="10.0 10.0 10.0"/>
-      </geometry>
-    </collision>
-  </link>
-  <joint name="joint_elbowR" type="revolute">
-    <origin
-      xyz="0.011176 -0.115 0.1917"
-      rpy="3.1416 0.058237 0" />
-    <parent link="shoulderR_link"/>
-    <child link="elbowR_link"/>
-    <axis xyz="0 1 0"/>
-    <limit
-      lower="-0.875"
-      upper="1.5708"
-      effort="10"
-      velocity="5" />
-  </joint>
-  <!-- ============================================================ -->
-  <!-- LEFT SHOULDER                                                  -->
-  <!-- ============================================================ -->
-  <link name="shoulderL_link">
-    <inertial>
-      <origin
-        xyz="-0.047911 -0.092283 0.044054"
-        rpy="0 0 0" />
-      <mass value="0.43205" />
-      <inertia
-        ixx="0.00097231"
-        ixy="-0.00015975"
-        ixz="0.00070474"
-        iyy="0.0015347"
-        iyz="0.00014689"
-        izz="0.0010908" />
-    </inertial>
-    <visual>
-      <origin xyz="0 0 0" rpy="0 0 0" />
-      <geometry>
-        <mesh
-          filename="package://human_urdf/meshes/shoulderL_link.STL"
-          scale="10.0 10.0 10.0"/>
-      </geometry>
-      <material name="">
-        <color rgba="0.79216 0.81961 0.93333 1" />
-      </material>
-    </visual>
-    <collision>
-      <origin xyz="0 0 0" rpy="0 0 0" />
-      <geometry>
-        <mesh
-          filename="package://human_urdf/meshes/shoulderL_link.STL"
-          scale="10.0 10.0 10.0"/>
-      </geometry>
-    </collision>
-  </link>
-  <joint name="joint_shoulderL" type="revolute">
-    <origin
-      xyz="-0.077756 0.025 -0.13145"
-      rpy="0 0 -1.5708" />
-    <parent link="base_link"/>
-    <child link="shoulderL_link"/>
-    <axis xyz="0 1 0"/>
-    <limit
-      lower="-1.5708"
-      upper="1.5708"
-      effort="10"
-      velocity="5" />
-  </joint>
-  <!-- ============================================================ -->
-  <!-- LEFT ELBOW                                                     -->
-  <!-- ============================================================ -->
-  <link name="elbowL_link">
-    <inertial>
-      <origin
-        xyz="-0.10017 -0.015 0.10211"
-        rpy="0 0 0" />
-      <mass value="0.47524" />
-      <inertia
-        ixx="0.0013144"
-        ixy="1.683E-12"
-        ixz="0.001148"
-        iyy="0.0024409"
-        iyz="1.4289E-12"
-        izz="0.0012704" />
-    </inertial>
-    <visual>
-      <origin xyz="0 0 0" rpy="0 0 0" />
-      <geometry>
-        <mesh
-          filename="package://human_urdf/meshes/elbowL_link.STL"
-          scale="10.0 10.0 10.0"/>
-      </geometry>
-      <material name="">
-        <color rgba="0.79216 0.81961 0.93333 1" />
-      </material>
-    </visual>
-    <collision>
-      <origin xyz="0 0 0" rpy="0 0 0" />
-      <geometry>
-        <mesh
-          filename="package://human_urdf/meshes/elbowL_link.STL"
-          scale="10.0 10.0 10.0"/>
-      </geometry>
-    </collision>
-  </link>
-  <joint name="joint_elbowL" type="revolute">
-    <origin
-      xyz="-0.14135 -0.115 0.12997"
-      rpy="0 0 3.1416" />
-    <parent link="shoulderL_link"/>
-    <child link="elbowL_link"/>
-    <axis xyz="0 1 0"/>
-    <limit
-      lower="-0.942"
-      upper="1.5708"
-      effort="10"
-      velocity="5" />
-  </joint>
-  <!-- ============================================================ -->
-  <!-- NECK                                                           -->
-  <!-- ============================================================ -->
-  <link name="neck_link">
-    <inertial>
-      <origin
-        xyz="0.0025028 0.04 -0.11501"
-        rpy="0 0 0" />
-      <mass value="7.8498" />
-      <inertia
-        ixx="0.0537"
-        ixy="2.9708E-18"
-        ixz="0.00099049"
-        iyy="0.043754"
-        iyz="-2.5878E-18"
-        izz="0.054124" />
-    </inertial>
-    <visual>
-      <origin xyz="0 0 0" rpy="0 0 0" />
-      <geometry>
-        <mesh
-          filename="package://human_urdf/meshes/neck_link.STL"
-          scale="10.0 10.0 10.0"/>
-      </geometry>
-      <material name="">
-        <color rgba="0.79216 0.81961 0.93333 1" />
-      </material>
-    </visual>
-    <collision>
-      <origin xyz="0 0 0" rpy="0 0 0" />
-      <geometry>
-        <mesh
-          filename="package://human_urdf/meshes/neck_link.STL"
-          scale="10.0 10.0 10.0"/>
-      </geometry>
-    </collision>
-  </link>
-  <joint name="joint_neck" type="revolute">
-    <origin
-      xyz="0.04 0.024699 -0.18935"
-      rpy="0 0 1.5708" />
-    <parent link="base_link"/>
-    <child link="neck_link"/>
-    <axis xyz="0 1 0"/>
-    <limit
-      lower="-1.5708"
-      upper="1.5708"
-      effort="10"
-      velocity="5" />
-  </joint>
-  <!-- ============================================================ -->
-  <!-- RIGHT WAIST                                                    -->
-  <!-- ============================================================ -->
-  <link name="waistR_link">
-    <inertial>
-      <origin
-        xyz="0.068854 -0.025 0.15762"
-        rpy="0 0 0" />
-      <mass value="1.3009" />
-      <inertia
-        ixx="0.0090303"
-        ixy="-1.1619E-09"
-        ixz="-0.0035584"
-        iyy="0.010576"
-        iyz="4.8063E-10"
-        izz="0.0024388" />
-    </inertial>
-    <visual>
-      <origin xyz="0 0 0" rpy="0 0 0" />
-      <geometry>
-        <mesh
-          filename="package://human_urdf/meshes/waistR_link.STL"
-          scale="10.0 10.0 10.0"/>
-      </geometry>
-      <material name="">
-        <color rgba="0.79216 0.81961 0.93333 1" />
-      </material>
-    </visual>
-    <collision>
-      <origin xyz="0 0 0" rpy="0 0 0" />
-      <geometry>
-        <mesh
-          filename="package://human_urdf/meshes/waistR_link.STL"
-          scale="10.0 10.0 10.0"/>
-      </geometry>
-    </collision>
-  </link>
-  <joint name="joint_waistR" type="revolute">
-    <origin
-      xyz="0.125 0.02366 0.21363"
-      rpy="0 0 -1.5708" />
-    <parent link="base_link"/>
-    <child link="waistR_link"/>
-    <axis xyz="0 1 0"/>
-    <limit
-      lower="-1.5708"
-      upper="1.5708"
-      effort="10"
-      velocity="5" />
-  </joint>
-  <!-- ============================================================ -->
-  <!-- RIGHT KNEE                                                     -->
-  <!-- ============================================================ -->
-  <link name="kneeR_link">
-    <inertial>
-      <origin
-        xyz="0.081339 -0.025 -0.12311"
-        rpy="0 0 0" />
-      <mass value="0.70121" />
-      <inertia
-        ixx="0.0027167"
-        ixy="-1.4134E-20"
-        ixz="0.0016128"
-        iyy="0.0037994"
-        iyz="2.6849E-20"
-        izz="0.0014034" />
-    </inertial>
-    <visual>
-      <origin xyz="0 0 0" rpy="0 0 0" />
-      <geometry>
-        <mesh
-          filename="package://human_urdf/meshes/kneeR_link.STL"
-          scale="10.0 10.0 10.0"/>
-      </geometry>
-      <material name="">
-        <color rgba="0.79216 0.81961 0.93333 1" />
-      </material>
-    </visual>
-    <collision>
-      <origin xyz="0 0 0" rpy="0 0 0" />
-      <geometry>
-        <mesh
-          filename="package://human_urdf/meshes/kneeR_link.STL"
-          scale="10.0 10.0 10.0"/>
-      </geometry>
-    </collision>
-  </link>
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
File: src/human_urdf/urdf/human_gazebo.xacro (robot description, xacro)
@@ -14,42 +14,42 @@
     </gazebo>
     <gazebo reference="camera_left_link">
-  <sensor name="left_eye_camera" type="camera">
-    <always_on>true</always_on>
-    <update_rate>30</update_rate>
-    <visualize>true</visualize>
-    <topic>left_camera/image_raw</topic>
-    <camera>
-      <horizontal_fov>1.047</horizontal_fov>
-      <image>
-        <width>640</width>
-        <height>480</height>
-        <format>R8G8B8</format>
-      </image>
-      <clip>
-        <near>0.05</near>
-        <far>50.0</far>
-      </clip>
-    </camera>
-  </sensor>
-</gazebo>
-<gazebo reference="camera_right_link">
-  <sensor name="right_eye_camera" type="camera">
-    <always_on>true</always_on>
-    <update_rate>30</update_rate>
-    <visualize>true</visualize>
-    <topic>right_camera/image_raw</topic>
-    <camera>
-      <horizontal_fov>1.047</horizontal_fov>
-      <image>
-        <width>640</width>
-        <height>480</height>
-        <format>R8G8B8</format>
-      </image>
-      <clip>
-        <near>0.05</near>
-        <far>50.0</far>
-      </clip>
-    </camera>
-  </sensor>
-</gazebo>
+        <sensor name="left_eye_camera" type="camera">
+        <always_on>true</always_on>
+        <update_rate>30</update_rate>
+        <visualize>true</visualize>
+        <topic>left_camera/image_raw</topic>
+        <camera>
+        <horizontal_fov>1.047</horizontal_fov>
+        <image>
+            <width>640</width>
+            <height>480</height>
+            <format>R8G8B8</format>
+        </image>
+        <clip>
+            <near>0.05</near>
+            <far>50.0</far>
+        </clip>
+        </camera>
+        </sensor>
+    </gazebo>
+    <gazebo reference="camera_right_link">
+        <sensor name="right_eye_camera" type="camera">
+            <always_on>true</always_on>
+            <update_rate>30</update_rate>
+            <visualize>true</visualize>
+            <topic>right_camera/image_raw</topic>
+            <camera>
+            <horizontal_fov>1.047</horizontal_fov>
+            <image>
+                <width>640</width>
+                <height>480</height>
+                <format>R8G8B8</format>
+            </image>
+            <clip>
+                <near>0.05</near>
+                <far>50.0</far>
+            </clip>
+            </camera>
+        </sensor>
+    </gazebo>
 </robot>

File: src/human_urdf/urdf/human_ros2_control.xacro (robot description, xacro)
@@ -99,4 +99,38 @@
             <state_interface name="velocity"/>
         </joint>
+                <!-- ========================= -->
+        <!-- LEFT GRIPPER              -->
+        <!-- ========================= -->
+        <joint name="joint_GripL1">
+            <command_interface name="position">
+                <param name="min">0.0</param>
+                <param name="max">1.5708</param>
+            </command_interface>
+            <state_interface name="position"/>
+            <state_interface name="velocity"/>
+        </joint>
+        <joint name="joint_GripL2">
+            <param name="mimic">joint_GripL1</param>
+            <param name="multiplier">-1</param>
+            <state_interface name="position"/>
+            <state_interface name="velocity"/>
+        </joint>
+        <!-- ========================= -->
+        <!-- RIGHT GRIPPER             -->
+        <!-- ========================= -->
+        <joint name="joint_GripR1">
+            <command_interface name="position">
+                <param name="min">0.0</param>
+                <param name="max">1.5708</param>
+            </command_interface>
+            <state_interface name="position"/>
+            <state_interface name="velocity"/>
+        </joint>
+        <joint name="joint_GripR2">
+            <param name="mimic">joint_GripR1</param>
+            <param name="multiplier">-1</param>
+            <state_interface name="position"/>
+            <state_interface name="velocity"/>
+        </joint>
     </ros2_control>
 </robot>
